Commit message: rtab-mapping working

File: urdf/my_robot.xacro (robot description, xacro)
@@ -1,5 +1,5 @@
 <?xml version='1.0'?>
 <robot name="my_robot" xmlns:xacro="http://www.ros.org/wiki/xacro">
-  <xacro:include filename="$(find udacity_bot)/urdf/my_robot.gazebo" />
+  <xacro:include filename="$(find map_my_world)/urdf/my_robot.gazebo" />
   <gazebo reference="left_wheel">
     <material>Gazebo/Blue</material>
@@ -23,7 +23,37 @@
     <origin xyz="0.2 0 0" rpy="0 0 0" />
     <parent link="chassis"/>
-    <child link="camera" />
+    <child link="camera_link" />
     <axis xyz="0 1 0"/>
   </joint>
+  <link name ='camera_link'>
+    <inertial>
+      <mass value="0.1"/>
+      <origin xyz="0 0 0" rpy="0 0 0"/>
+      <inertia
+          ixx="1e-6" ixy="0" ixz="0"
+          iyy="1e-6" iyz="0"
+          izz="1e-6"
+      />
+    </inertial>
+    <collision name='collision_camera'>
+      <origin xyz="0 0 0" rpy="0 0 0"/>
+      <geometry>
+        <box size ="0.05 0.05 0.05"/>
+      </geometry>
+    </collision>
+    <visual name='camera_visual'>
+      <origin xyz="0 0 0" rpy="0 0 0"/>
+      <geometry>
+        <box size ="0.05 0.05 0.05"/>
+      </geometry>
+    </visual>
+   </link>
+  <joint name="camera_optical_joint" type="fixed">
+    <origin xyz="0 0 0" rpy="-1.5707 0 -1.5707"/>
+    <parent link="camera_link"/>
+    <child link="camera_link_optical"/>
+  </joint>
+  <link name="camera_link_optical">
+  </link>
   <joint name="hokuyo_joint" type="fixed">
     <origin xyz="0.15 0 0.08" rpy="0 0 0" />
@@ -48,27 +78,4 @@
     <dynamics damping="1.0" friction="1.0"/>
   </joint>
-  <link name="camera">
-    <inertial>
-      <mass value="0.1"/>
-      <origin xyz="0 0 0" rpy="0 0 0"/>
-      <inertia
-        ixx="1e-6" ixy="0.0" ixz="0.0"
-        iyy="1e-6" iyz="0.0"
-        izz="1e-6"
-      />
-    </inertial>
-    <collision>
-      <origin xyz="0 0 0" rpy="0 0 0"/>
-      <geometry>
-        <box size="0.05 0.05 0.05"/>
-      </geometry>
-    </collision>
-    <visual>
-      <origin xyz="0 0 0" rpy="0 0 0"/>
-      <geometry>
-        <box size="0.05 0.05 0.05"/>
-      </geometry>
-    </visual>
-  </link>
   <link name="hokuyo">
     <inertial>
@@ -90,5 +97,5 @@
       <origin xyz="0 0 0" rpy="0 0 0"/>
       <geometry>
-        <mesh filename="package://udacity_bot/meshes/hokuyo.dae"/>
+        <mesh filename="package://map_my_world/meshes/hokuyo.dae"/>
       </geometry>
     </visual>
